File: HSLinkCompact_v1.3.1/HSLinkPro.kicad_pcb (KiCad board)
At the start: 4 copper layers, 44 x 44 mm, 155 parts, among them J1 IDC 2x10p 夹板, J2 USB_C_Receptacle_USB2.0, J3 Header 1.27 4P, Q2 SS8050, Q3 AO3401, Q4 SS8050, Q5 SS8050, Q6 AO3401, Q7 AO3401, Q8 SS8050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

Commit message: 降低工艺需求
Parts:
- moved R15 1.52 mm to (102.5, 91.0), turned to 0 degrees
- moved R32 1.05 mm to (127.7, 106.3)
- moved R33 1.05 mm to (127.7, 107.4)
- moved R14 0.74 mm to (102.5, 92.1), turned to 0 degrees
- moved R23 0.51 mm to (110.2, 97.0)
- moved R22 0.51 mm to (109.1, 97.0)
- moved C13 0.40 mm to (115.7, 106.7)
- moved C3 0.38 mm to (119.3, 106.7)
- moved C6 0.38 mm to (118.3, 106.7)
- moved U3 0.38 mm to (113.1, 88.3)
- turned R36 to 180 degrees
Routing:
- net GND: track 20.6 -> 24.9 mm, vias 162 -> 163
- net /MCU/WS2812: track 62.4 -> 59.2 mm
- net Net-(U12-B): track 16.6 -> 19.8 mm
- net Net-(U11-B): track 15.0 -> 18.0 mm
- net /PORT_EN: track 18.5 -> 20.5 mm
- net Net-(U4-B): track 18.6 -> 20.3 mm
- net /MCU/SWCLK/TCK: track 35.2 -> 36.7 mm
- net Net-(U2-B): track 23.3 -> 24.9 mm
- net Net-(U3-B): track 21.7 -> 23.1 mm
- net Net-(J2-CC2): track 13.4 -> 14.6 mm
- net /MCU/SPI_CS: track 16.2 -> 15.1 mm
- net Net-(U5-B): track 26.1 -> 27.1 mm
- net /MCU/TRANS_PWM: track 38.4 -> 39.3 mm, vias 2 -> 4
- net /MCU/UART_EN#: track 12.4 -> 11.6 mm
- net /UART_RTS: track 9.15 -> 8.53 mm
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