File: HSLinkPro_v1.2.1/HSLinkPro.kicad_pcb (KiCad board)
At the start: 4 copper layers, 26 x 35 mm, 130 parts, among them J1 IDC 2x10p 夹板, J2 USB_C_Receptacle_USB2.0, J3 Header 1.27 4P, Q1 2N7002, SW1 1TS028A-1900-0600-CT, U1 HPM5301IEG1, U10 TLV62568DRL, U11 SN74LVC1T45DCK, U12 SN74LVC1T45DCK, U13 LMV321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

Commit message: fix: 1.2.1 修复UART RX未上拉问题
Parts:
- added R19: 100k, Resistor_SMD:R_0402_1005Metric, F.Cu at (116.8, 59.2)
Routing:
- net TRANS_VCC_OUT: track 8.47 -> 37.7 mm, vias 2 -> 3
- net /Interface /UART_RX: track 4.05 -> 7.81 mm, vias 1 -> 2
